Commit message: remove from lifecycle, new urdf

File: nav2_bringup/urdf/robotino.urdf (robot description, URDF)
Before this commit: robot robot, 21 links, 20 joints
Joints:
- joint joint_gripper_x_dyn_to_gripper_y_origin: parent gripper_x_dyn -> gripper_x_origin
- joint joint_gripper_y_dyn_to_cam_base: parent gripper_y_dyn -> gripper_y_origin
- joint joint_gripper_y_dyn_to_cam_gripper: parent gripper_y_dyn -> gripper_y_origin
- joint joint_gripper_y_dyn_to_gripper_z_origin: parent gripper_y_dyn -> gripper_y_origin
- joint joint_gripper_z_dyn_to_gripper: parent gripper_z_dyn -> gripper_z_origin
